File: PCB/ESP8285_WiFi.sch (KiCad schematic (older format))
At the start: 0 parts

Commit message: Progress
Datasheets added for regulators, regulators chosen, more datasheets
ralted to Zync 7000 added. Memory module chose footprint created and
datasheet added. Schematic work in progress. Project is slow going do to
th sheer amount of documenation to absorb on the Zync and makign high
pin count BGAs is tedious. More to follow soon.
Parts:
- added C19, C21: CL05C090CB5NNNC, PCB_Footprints:C0402, symbol CL05C090CB5NNNC
- added C20, C22, C23, C24, C25, C26, C27, C28: CL05B104JP5NNNC, PCB_Footprints:C0402, symbol CL05B104JP5NNNC
- added C29: 600L5R6BT200T, PCB_Footprints:C0402, symbol 600L5R6BT200T
- added LED4: LTST-C193TBKT-5A, PCB_Footprints:LED0603, symbol LTST-C193TBKT-5A
- added R20, R21: RC1005F102CS, PCB_Footprints:R0402, symbol RC1005F102CS
- added R22, R23: RC1005F123CS, PCB_Footprints:R0402, symbol RC1005F123CS
- added R24: RC1005F103CS, PCB_Footprints:R0402, symbol RC1005F103CS
- added SW2: B3U-1000P, PCB_Footprints:B3U-1000P, symbol B3U-1000P
- added T1: 1909763-1, PCB_Footprints:1909763-1, symbol 1909763-1
- added U4: ESP8285, PCB_Footprints:ESP8285, symbol ESP8285
- added X3: FA-128_26.0000MF10Z-AC3, PCB_Footprints:FA-128_26.0000MF10Z-AC3, symbol FA-128_26.0000MF10Z-AC3
Connections:
- new net: LED4.1, R21.2
- new net: R21.1, U4.18 (SD_DATA_2)
- new net: C19.1, U4.27 (XTAL_OUT), X3.1
- new net: C21.1, U4.28 (XTAL_IN), X3.3
- new net: R22.1, U4.7 (CHIP_EN)
- new net: R23.2, U4.31 (RES12K)
- new net +3V3: C20.1, C22.1, C23.1, C24.1, C26.1, C27.1, C28.1, R20.2, R22.2, R24.1, U4.1 (VDDA), U4.11 (VDDPST), U4.17 (VDDPST), U4.29 (VDDD), U4.3 (VDD3P3), U4.30 (VDDA), U4.4 (VDD3P3)
- new net ANT_UM: C29.2, T1.1
- new net ESPTOST_BOOT0: U4.22 (SD_DATA_0)
- new net ESPTOST_BOOT1: U4.23 (SD_DATA_1)
- new net ESP_PGM_MODE: R24.2, U4.15 (GPIO0)
- new net ESP_ST_RST: U4.24 (GPIO5)
- new net ESP_URX: U4.26 (U0_TXD)
- new net ESP_UTX: U4.25 (U0_RXD)
- new net GND: C19.2, C20.2, C21.2, C22.2, C23.2, C24.2, C25.2, C26.2, C27.2, C28.2, LED4.2, R23.1, SW2.1, T1.2, U4.33 (GND), X3.2, X3.4
- new net LNA: C29.1, U4.2 (LNA)
- new net STM_ESP_RST: C25.1, R20.1, SW2.2, U4.32 (EXT_RSTB)
Other:
- note added: "ESP8285 WiFi Radio"
