File: PCB/_saved_SoC_PMIC.sch (KiCad schematic (older format))
At the start: 19 parts

Commit message: PMIC
PMIC components chosen with symbols/footprints all created. See
hydroPWNics footprints lib for details. Currently working on PMIC
schematic everything else comes next.
Parts:
- added Q? (x2): FDMC7660, PCB_Footprints:FDMC7660, symbol FDMC7660
Connections:
- wire segments 48 -> 57
Changed lines of the file:
@@
 	9350 5050 10975 5050
 Wire Wire Line
-	9350 4100 10975 4100
+	9350 4100 9350 4100
 Text Notes 5875 900  0    197  ~ 39
 System PMIC: TPS659118A2ZRCT
@@
 	6750 6500 6750 6600
 Wire Wire Line
-	6750 6500 4750 6500
-Wire Wire Line
-	6750 5750 4750 5750
-Wire Wire Line
-	6750 4900 4750 4900
+	4750 6500 6750 6500
+Wire Wire Line
+	4750 5750 6750 5750
+Wire Wire Line
+	4750 4900 6750 4900
 $Comp
 L CL10A225KQ8NNNC C?
@@
 	1    0    0    -1
 $EndComp
+$Comp
+L FDMC7660 Q?
+U 1 1 588C9F08
+P 11500 3650
+F 0 "Q?" H 11725 3750 60  0000 C CNN
+F 1 "FDMC7660" H 11900 3650 60  0000 C CNN
+F 2 "PCB_Footprints:FDMC7660" H 12800 6150 60  0001 C CNN
+F 3 "https://www.fairchildsemi.com/datasheets/FD/FDMC7660.pdf" H 13100 6350 60  0001 C CNN
+F 4 "0.67500 @ 3000" H 12600 6650 60  0001 C CNN "Cost"
+F 5 "21 Jan 2017" H 12650 6550 60  0001 C CNN "Date Created "
+F 6 "21 Jan 2017" H 12700 6000 60  0001 C CNN "Date Modified"
+F 7 "Adam Vadala-Roth" H 12600 6450 60  0001 C CNN "Designer"
+F 8 "0.4mm" H 12650 6250 60  0001 C CNN "Height"
+F 9 "Yes" H 12650 6750 60  0001 C CNN "RHoS?"
+F 10 "Fairchild/ON Semiconductor" H 12700 5900 60  0001 C CNN "MFR"
+F 11 "FDMC7660" H 11750 4900 60  0001 C CNN "MFR#"
+F 12 "SMT/SMD" H 11850 5000 60  0001 C CNN "Mounting"
+F 13 "2" H 11950 5100 60  0001 C CNN "Pin Count#"
+F 14 "Active" H 12050 5200 60  0001 C CNN "Status"
+F 15 "N/A" H 12150 5300 60  0001 C CNN "Tolerance"
+F 16 "MOSFET N-CH 30V 20A 8-PQFN" H 12250 5400 60  0001 C CNN "Type"
+F 17 "30V" H 12350 5500 60  0001 C CNN "Voltage"
+F 18 "N/A" H 12450 5600 60  0001 C CNN "Wattage"
+F 19 "N/A" H 12550 5700 60  0001 C CNN "Component-Value"
+F 20 "N-Channel 30V 20A (Ta), 40A (Tc) 2.3W (Ta), 41W (Tc) Surface Mount 8-PQFN (3.3x3.3), Power33" H 12650 5800 60  0001 C CNN "Description"
+	1    11500 3650
+	1    0    0    -1
+$EndComp
+Wire Wire Line
+	9350 3700 11200 3700
+$Comp
+L FDMC7660 Q?
+U 1 1 588CA987
+P 11950 4200
+F 0 "Q?" H 12175 4300 60  0000 C CNN
+F 1 "FDMC7660" H 12350 4200 60  0000 C CNN
+F 2 "PCB_Footprints:FDMC7660" H 13250 6700 60  0001 C CNN
+F 3 "https://www.fairchildsemi.com/datasheets/FD/FDMC7660.pdf" H 13550 6900 60  0001 C CNN
+F 4 "0.67500 @ 3000" H 13050 7200 60  0001 C CNN "Cost"
+F 5 "21 Jan 2017" H 13100 7100 60  0001 C CNN "Date Created "
+F 6 "21 Jan 2017" H 13150 6550 60  0001 C CNN "Date Modified"
+F 7 "Adam Vadala-Roth" H 13050 7000 60  0001 C CNN "Designer"
+F 8 "0.4mm" H 13100 6800 60  0001 C CNN "Height"
+F 9 "Yes" H 13100 7300 60  0001 C CNN "RHoS?"
+F 10 "Fairchild/ON Semiconductor" H 13150 6450 60  0001 C CNN "MFR"
+F 11 "FDMC7660" H 12200 5450 60  0001 C CNN "MFR#"
+F 12 "SMT/SMD" H 12300 5550 60  0001 C CNN "Mounting"
+F 13 "2" H 12400 5650 60  0001 C CNN "Pin Count#"
+F 14 "Active" H 12500 5750 60  0001 C CNN "Status"
+F 15 "N/A" H 12600 5850 60  0001 C CNN "Tolerance"
+F 16 "MOSFET N-CH 30V 20A 8-PQFN" H 12700 5950 60  0001 C CNN "Type"
+F 17 "30V" H 12800 6050 60  0001 C CNN "Voltage"
+F 18 "N/A" H 12900 6150 60  0001 C CNN "Wattage"
+F 19 "N/A" H 13000 6250 60  0001 C CNN "Component-Value"
+F 20 "N-Channel 30V 20A (Ta), 40A (Tc) 2.3W (Ta), 41W (Tc) Surface Mount 8-PQFN (3.3x3.3), Power33" H 13100 6350 60  0001 C CNN "Description"
+	1    11950 4200
+	1    0    0    -1
+$EndComp
+Wire Wire Line
+	9350 4250 11650 4250
+Wire Wire Line
+	9350 4100 9350 4175
+Wire Wire Line
+	11600 4175 9350 4175
+Wire Wire Line
+	11600 3900 11600 4175
+Connection ~ 11600 4100
+Connection ~ 11600 4000
+Wire Wire Line
+	12050 3850 12050 3775
+Wire Wire Line
+	12050 3775 11700 3775
+Wire Wire Line
+	11700 3775 11700 3900
+Wire Wire Line
+	11700 3900 11600 3900
 $EndSCHEMATC
