File: PCB/Memory.sch (KiCad schematic (older format))
At the start: 0 parts

Commit message: Progress
Datasheets added for regulators, regulators chosen, more datasheets
ralted to Zync 7000 added. Memory module chose footprint created and
datasheet added. Schematic work in progress. Project is slow going do to
th sheer amount of documenation to absorb on the Zync and makign high
pin count BGAs is tedious. More to follow soon.
Parts:
- added U? (x2): MT41K128M8DA-107:J, PCB_Footprints:MT41K128M8DA_107_J, symbol MT41K128M8DA-107:J
Connections:
- net labels added: GND, MEM_DATA_BUS, RAM_A3_NC, RAM_F1_NC, RAM_F9_NC, RAM_H1_NC, RAM_H9_NC, RAM_J7_NC, RAM_N7_NC
- wire segments 0 -> 25
Changed lines of the file:
@@
 LIBS:HydroPWNics_Lib
 LIBS:OnHand-Components-Sym
+LIBS:ZyncMV-cache
 EELAYER 25 0
 EELAYER END
 $Descr A4 11693 8268
 encoding utf-8
-Sheet 6 11
+Sheet 6 8
 Title ""
 Date ""
@@
 Comment4 ""
 $EndDescr
+$Comp
+L MT41K128M8DA-107:J U?
+U 1 1 587AE94B
+P 4400 2350
+F 0 "U?" H 4375 3447 60  0000 C CNN
+F 1 "MT41K128M8DA-107:J" H 4375 3341 60  0000 C CNN
+F 2 "PCB_Footprints:MT41K128M8DA_107_J" H 5825 4275 60  0001 C CNN
+F 3 "http://www.micron.com/~/media/documents/products/data-sheet/dram/ddr3/1gb_1_35v_ddr3l.pdf" H 6025 4400 60  0001 C CNN
+F 4 "3.20400 @ 250" H 4450 3325 60  0001 C CNN "Cost"
+F 5 "7 Jan 2017" H 4475 3425 60  0001 C CNN "Date Created"
+F 6 "7 Jan 2017" H 4575 3525 60  0001 C CNN "Date Modified"
+F 7 "Adam Vadala-Roth" H 4675 3625 60  0001 C CNN "Designer"
+F 8 "0.8mm" H 4775 3725 60  0001 C CNN "Height"
+F 9 "Yes" H 4875 3825 60  0001 C CNN "RhoS?"
+F 10 "Micron" H 4975 3925 60  0001 C CNN "MFR"
+F 11 "MT41K128M8DA-107:J" H 5075 4025 60  0001 C CNN "MFR#"
+F 12 "SMT/SMD" H 5175 4125 60  0001 C CNN "Mounting"
+F 13 "78" H 5275 4225 60  0001 C CNN "Pin Count#"
+F 14 "Active" H 5375 4325 60  0001 C CNN "Status"
+F 15 "N/A" H 5475 4425 60  0001 C CNN "Tolerance"
+F 16 "DDR3L SDRAM Module" H 5575 4525 60  0001 C CNN "Type"
+F 17 "N/A" H 5675 4625 60  0001 C CNN "Voltage"
+F 18 "N/A" H 5650 3950 60  0001 C CNN "Wattage"
+F 19 "N/A" H 5750 4050 60  0001 C CNN "Component-Value"
+F 20 "IC SDRAM 1GBIT 933MHZ 78FBGA" H 5850 4150 60  0001 C CNN "Description"
+	1    4400 2350
+	1    0    0    -1
+$EndComp
+$Comp
+L MT41K128M8DA-107:J U?
+U 2 1 587AEA02
+P 4250 5500
+F 0 "U?" H 3850 6300 60  0000 C CNN
+F 1 "MT41K128M8DA-107:J" H 4250 4350 60  0000 C CNN
+F 2 "PCB_Footprints:MT41K128M8DA_107_J" H 5675 7425 60  0001 C CNN
+F 3 "http://www.micron.com/~/media/documents/products/data-sheet/dram/ddr3/1gb_1_35v_ddr3l.pdf" H 5875 7550 60  0001 C CNN
+F 4 "3.20400 @ 250" H 4300 6475 60  0001 C CNN "Cost"
+F 5 "7 Jan 2017" H 4325 6575 60  0001 C CNN "Date Created"
+F 6 "7 Jan 2017" H 4425 6675 60  0001 C CNN "Date Modified"
+F 7 "Adam Vadala-Roth" H 4525 6775 60  0001 C CNN "Designer"
+F 8 "0.8mm" H 4625 6875 60  0001 C CNN "Height"
+F 9 "Yes" H 4725 6975 60  0001 C CNN "RhoS?"
+F 10 "Micron" H 4825 7075 60  0001 C CNN "MFR"
+F 11 "MT41K128M8DA-107:J" H 4925 7175 60  0001 C CNN "MFR#"
+F 12 "SMT/SMD" H 5025 7275 60  0001 C CNN "Mounting"
+F 13 "78" H 5125 7375 60  0001 C CNN "Pin Count#"
+F 14 "Active" H 5225 7475 60  0001 C CNN "Status"
+F 15 "N/A" H 5325 7575 60  0001 C CNN "Tolerance"
+F 16 "DDR3L SDRAM Module" H 5425 7675 60  0001 C CNN "Type"
+F 17 "N/A" H 5525 7775 60  0001 C CNN "Voltage"
+F 18 "N/A" H 5500 7100 60  0001 C CNN "Wattage"
+F 19 "N/A" H 5600 7200 60  0001 C CNN "Component-Value"
+F 20 "IC SDRAM 1GBIT 933MHZ 78FBGA" H 5700 7300 60  0001 C CNN "Description"
+	2    4250 5500
+	1    0    0    -1
+$EndComp
+Wire Wire Line
+	5200 3700 5800 3700
+Wire Wire Line
+	5800 3800 5200 3800
+Wire Wire Line
+	5800 3900 5200 3900
+Wire Wire Line
+	5800 4000 5200 4000
+Wire Wire Line
+	5800 4100 5200 4100
+Wire Wire Line
+	5800 4200 5200 4200
+Wire Wire Line
+	5800 4300 5200 4300
+Text Label 5250 3700 0    60   ~ 0
+RAM_A3_NC
+Text Label 5250 3800 0    60   ~ 0
+RAM_F1_NC
+Text Label 5250 3900 0    60   ~ 0
+RAM_H1_NC
+Text Label 5250 4000 0    60   ~ 0
+RAM_F9_NC
+Text Label 5250 4100 0    60   ~ 0
+RAM_H9_NC
+Text Label 5250 4200 0    60   ~ 0
+RAM_J7_NC
+Text Label 5250 4300 0    60   ~ 0
+RAM_N7_NC
+Wire Wire Line
+	3550 4800 3550 4900
+Wire Wire Line
+	3550 4800 2850 4800
+Wire Wire Line
+	5000 4800 5000 4900
+Wire Wire Line
+	5000 4900 5000 5000
+Wire Wire Line
+	5000 5000 5000 5100
+Wire Wire Line
+	5000 5100 5000 5200
+Wire Wire Line
+	5000 5200 5000 5450
+Wire Wire Line
+	5000 5450 5000 5550
+Wire Wire Line
+	5000 5550 5000 5650
+Wire Wire Line
+	5000 5650 5000 5750
+Wire Wire Line
+	5000 5750 5000 5850
+Wire Wire Line
+	5000 5850 5000 5950
+Wire Wire Line
+	5000 5950 5000 6050
+Wire Wire Line
+	5000 6050 5000 6150
+Wire Wire Line
+	5000 6150 5000 6250
+Wire Wire Line
+	5000 6250 5000 6350
+Wire Wire Line
+	5000 6350 5000 6450
+Wire Wire Line
+	5000 6450 5000 6550
+Connection ~ 5000 4900
+Connection ~ 5000 5000
+Connection ~ 5000 5100
+Connection ~ 5000 5200
+Connection ~ 5000 5450
+Connection ~ 5000 5550
+Connection ~ 5000 5650
+Connection ~ 5000 5750
+Connection ~ 5000 5850
+Connection ~ 5000 5950
+Connection ~ 5000 6050
+Connection ~ 5000 6150
+Connection ~ 5000 6250
+Connection ~ 5000 6350
+Connection ~ 5000 6450
+$Comp
+L GND #PWR?
+U 1 1 587AF98A
+P 5000 6550
+F 0 "#PWR?" H 5000 6300 50  0001 C CNN
+F 1 "GND" H 5005 6377 50  0000 C CNN
+F 2 "" H 5000 6550 50  0000 C CNN
+F 3 "" H 5000 6550 50  0000 C CNN
+	1    5000 6550
+	1    0    0    -1
+$EndComp
+Wire Bus Line
+	7250 1600 7250 1600
+Wire Bus Line
+	7250 1600 7250 1700
+Wire Bus Line
+	7250 1700 7250 1800
+Wire Bus Line
+	7250 1800 7250 1900
+Wire Bus Line
+	7250 1900 7250 2000
+Wire Bus Line
+	7250 2000 7250 2100
+Wire Bus Line
+	7250 2100 7250 2200
+Wire Bus Line
+	7250 2200 7250 2300
+Wire Bus Line
+	7250 2300 7250 2350
+Wire Bus Line
+	7250 2350 10250 2350
+Entry Bus Bus
+	7150 1500 7250 1600
+Entry Bus Bus
+	7150 1600 7250 1700
+Entry Bus Bus
+	7150 1700 7250 1800
+Entry Bus Bus
+	7150 1800 7250 1900
+Entry Bus Bus
+	7150 1900 7250 2000
+Entry Bus Bus
+	7150 2200 7250 2300
+Entry Bus Bus
+	7150 2100 7250 2200
+Entry Bus Bus
+	7150 2000 7250 2100
+Text HLabel 10250 2350 2    60   BiDi ~ 0
+MEM_DATA_BUS
 $EndSCHEMATC

Commit message: License
License added some progress on the memory
Parts:
- added R? (x25): ERA-2AEB510X, PCB_Footprints:R0402, symbol ERA-2AEB510X
Connections:
- wire segments 25 -> 58
Other:
- note added: "MT41K128M8DA-107:J 1GB DDR3L Memory"
- note added: "Place impedance matching\n resistors close to Zync SoC"

Commit message: PMIC
Switching to a PMIC topology since its a better solution for powering
the diverse set of hardware on the ZyncMV. The PMIC can be controlled by
the processor and shut down the device like a regular SBC. The PMIC als
has all the appropraite voltages for the memory and enough current to
support it. Additional regulartors still mayb required for supplying the
image sensor and most defintiely the light sources.
Connections:
- net labels added: MEM_ADDR_BUS
- wire segments 58 -> 83
Changed lines of the file:
@@
 	4525 4825 3825 4825
 Wire Wire Line
-	5975 4825 5975 6575
+	5975 4825 5975 4925
+Wire Wire Line
+	5975 4925 5975 5025
+Wire Wire Line
+	5975 5025 5975 5125
+Wire Wire Line
+	5975 5125 5975 5225
+Wire Wire Line
+	5975 5225 5975 5475
+Wire Wire Line
+	5975 5475 5975 5575
+Wire Wire Line
+	5975 5575 5975 5675
+Wire Wire Line
+	5975 5675 5975 5775
+Wire Wire Line
+	5975 5775 5975 5875
+Wire Wire Line
+	5975 5875 5975 5975
+Wire Wire Line
+	5975 5975 5975 6075
+Wire Wire Line
+	5975 6075 5975 6175
+Wire Wire Line
+	5975 6175 5975 6275
+Wire Wire Line
+	5975 6275 5975 6375
+Wire Wire Line
+	5975 6375 5975 6475
+Wire Wire Line
+	5975 6475 5975 6575
 Connection ~ 5975 4925
 Connection ~ 5975 5025
@@
 $EndComp
 Wire Bus Line
-	8225 1625 8225 2375
+	8225 1625 8225 1725
+Wire Bus Line
+	8225 1725 8225 1825
+Wire Bus Line
+	8225 1825 8225 1925
+Wire Bus Line
+	8225 1925 8225 2025
+Wire Bus Line
+	8225 2025 8225 2125
+Wire Bus Line
+	8225 2125 8225 2225
+Wire Bus Line
+	8225 2225 8225 2325
+Wire Bus Line
+	8225 2325 8225 2375
 Entry Bus Bus
 	8125 1525 8225 1625
@@
 	8225 2375 10225 2375
 Wire Bus Line
-	2750 1625 2750 3025
-Wire Bus Line
-	2750 3025 1225 3025
-Text HLabel 1225 3025 0    60   BiDi ~ 0
-MEM_DATA_BUS
+	2750 1625 2750 1725
+Wire Bus Line
+	2750 1725 2750 1825
+Wire Bus Line
+	2750 1825 2750 1925
+Wire Bus Line
+	2750 1925 2750 2025
+Wire Bus Line
+	2750 2025 2750 2125
+Wire Bus Line
+	2750 2125 2750 2225
+Wire Bus Line
+	2750 2225 2750 2325
+Wire Bus Line
+	2750 2325 2750 2425
+Wire Bus Line
+	2750 2425 2750 2525
+Wire Bus Line
+	2750 2525 2750 2625
+Wire Bus Line
+	2750 2625 2750 2725
+Wire Bus Line
+	2750 2725 2750 2825
+Wire Bus Line
+	2750 2825 2750 2925
+Wire Bus Line
+	2750 2925 2750 3125
+Wire Bus Line
+	2750 3125 2750 3225
+Wire Bus Line
+	2750 3225 2750 3325
+Wire Bus Line
+	2750 3325 2750 3450
+Wire Bus Line
+	2750 3450 1275 3450
+Text HLabel 1275 3450 0    60   BiDi ~ 0
+MEM_ADDR_BUS
 Text Notes 2975 1425 0    60   ~ 0
 Place impedance matching\n resistors close to Zync SoC
@@
 Place impedance matching\n resistors close to Zync SoC
 Wire Wire Line
-	4525 5775 4525 6575
+	4525 5775 4525 5875
+Wire Wire Line
+	4525 5875 4525 5975
+Wire Wire Line
+	4525 5975 4525 6075
+Wire Wire Line
+	4525 6075 4525 6175
+Wire Wire Line
+	4525 6175 4525 6275
+Wire Wire Line
+	4525 6275 4525 6375
+Wire Wire Line
+	4525 6375 4525 6475
+Wire Wire Line
+	4525 6475 4525 6575
 Connection ~ 4525 5875
 Connection ~ 4525 5975
@@
 Text Notes 3025 950  0    197  ~ 39
 MT41K128M8DA-107:J 1GB DDR3L Memory
+Wire Wire Line
+	2850 3125 3225 3125
+Wire Wire Line
+	2850 3225 3225 3225
+Entry Bus Bus
+	2750 3125 2850 3025
+Entry Bus Bus
+	2750 3225 2850 3125
+Entry Bus Bus
+	2750 3325 2850 3225
+Wire Wire Line
+	2850 3025 3225 3025
 $EndSCHEMATC

Commit message: Power
Power topology change. Power system schematic spans 3 pages. two for the
PMIC that supplies the SoC and the DDR3L and an addional page covering
input stage and DCDC regulators for other voltages, particularly for the
off board lighting module.
Connections:
- wire segments 83 -> 61
Changed lines of the file:
@@
 $Descr A4 11693 8268
 encoding utf-8
-Sheet 6 8
+Sheet 5 9
 Title ""
 Date "2016-12-23"
@@
 	4525 4825 3825 4825
 Wire Wire Line
-	5975 4825 5975 4925
-Wire Wire Line
-	5975 4925 5975 5025
-Wire Wire Line
-	5975 5025 5975 5125
-Wire Wire Line
-	5975 5125 5975 5225
-Wire Wire Line
-	5975 5225 5975 5475
-Wire Wire Line
-	5975 5475 5975 5575
-Wire Wire Line
-	5975 5575 5975 5675
-Wire Wire Line
-	5975 5675 5975 5775
-Wire Wire Line
-	5975 5775 5975 5875
-Wire Wire Line
-	5975 5875 5975 5975
-Wire Wire Line
-	5975 5975 5975 6075
-Wire Wire Line
-	5975 6075 5975 6175
-Wire Wire Line
-	5975 6175 5975 6275
-Wire Wire Line
-	5975 6275 5975 6375
-Wire Wire Line
-	5975 6375 5975 6475
-Wire Wire Line
-	5975 6475 5975 6575
+	5975 4825 5975 6575
 Connection ~ 5975 4925
 Connection ~ 5975 5025
@@
 $EndComp
 Wire Bus Line
-	8225 1625 8225 1725
-Wire Bus Line
-	8225 1725 8225 1825
-Wire Bus Line
-	8225 1825 8225 1925
-Wire Bus Line
-	8225 1925 8225 2025
-Wire Bus Line
-	8225 2025 8225 2125
-Wire Bus Line
-	8225 2125 8225 2225
-Wire Bus Line
-	8225 2225 8225 2325
-Wire Bus Line
-	8225 2325 8225 2375
+	8225 1625 8225 2375
 Entry Bus Bus
 	8125 1525 8225 1625
@@
 	8225 2375 10225 2375
 Wire Bus Line
-	2750 1625 2750 1725
-Wire Bus Line
-	2750 1725 2750 1825
-Wire Bus Line
-	2750 1825 2750 1925
-Wire Bus Line
-	2750 1925 2750 2025
-Wire Bus Line
-	2750 2025 2750 2125
-Wire Bus Line
-	2750 2125 2750 2225
-Wire Bus Line
-	2750 2225 2750 2325
-Wire Bus Line
-	2750 2325 2750 2425
-Wire Bus Line
-	2750 2425 2750 2525
-Wire Bus Line
-	2750 2525 2750 2625
-Wire Bus Line
-	2750 2625 2750 2725
-Wire Bus Line
-	2750 2725 2750 2825
-Wire Bus Line
-	2750 2825 2750 2925
-Wire Bus Line
-	2750 2925 2750 3125
-Wire Bus Line
-	2750 3125 2750 3225
-Wire Bus Line
-	2750 3225 2750 3325
-Wire Bus Line
-	2750 3325 2750 3450
+	2750 1625 2750 3450
 Wire Bus Line
 	2750 3450 1275 3450
@@
 Place impedance matching\n resistors close to Zync SoC
 Wire Wire Line
-	4525 5775 4525 5875
-Wire Wire Line
-	4525 5875 4525 5975
-Wire Wire Line
-	4525 5975 4525 6075
-Wire Wire Line
-	4525 6075 4525 6175
-Wire Wire Line
-	4525 6175 4525 6275
-Wire Wire Line
-	4525 6275 4525 6375
-Wire Wire Line
-	4525 6375 4525 6475
-Wire Wire Line
-	4525 6475 4525 6575
+	4525 5775 4525 6575
 Connection ~ 4525 5875
 Connection ~ 4525 5975

Commit message: DDR3L
major progress on DDR3L schematic. Still need to edit bus enries and
make control signals their own entry each.
Parts:
- added C? (x14): CL05A104JO5NNNC, PCB_Footprints:C0402, symbol CL05A104JO5NNNC
- added R? (x13): ERA-2AEB510X, PCB_Footprints:R0402, symbol ERA-2AEB510X
- added R?: ERJ-2RKF2400X, PCB_Footprints:R0402, symbol ERJ-2RKF2400X
Connections:
- net labels added: +1V35, CTRL_SIG_BUS, DDR3L_A0, DDR3L_A1, DDR3L_A10, DDR3L_A11, DDR3L_A12, DDR3L_A13, DDR3L_A2, DDR3L_A3, DDR3L_A4, DDR3L_A5, DDR3L_A6, DDR3L_A7, DDR3L_A8, DDR3L_A9, DDR3L_BA0, DDR3L_BA1, DDR3L_BA2, DDR3L_BA[1..17], DDR3L_CAS#, DDR3L_CK, DDR3L_CK#, DDR3L_CKE, DDR3L_CS#, DDR3L_D0, DDR3L_D1, DDR3L_D2, DDR3L_D3, DDR3L_D4, DDR3L_D5, DDR3L_D6, DDR3L_D7, DDR3L_DQS, DDR3L_DQS#, DDR3L_ODT, DDR3L_RAS#, DDR3L_RESET#, DDR3L_TDQS, DDR3L_TDQS#, DDR3L_VREF, DDR3L_WE#
- wire segments 61 -> 142
Other:
- moved on the sheet: R?

Commit message: PMIC
PMIC components chosen with symbols/footprints all created. See
hydroPWNics footprints lib for details. Currently working on PMIC
schematic everything else comes next.
Parts:
- removed U? (x2): MT41K128M8DA-107:J, PCB_Footprints:MT41K128M8DA_107_J, symbol MT41K128M8DA-107:J
- added U? (x2): MT41K512M8DA-107-XIT:P, PCB_Footprints:MT41K128M8DA_107_J, symbol MT41K512M8DA-107-XIT:P
Connections:
- wire segments 142 -> 94

Commit message: Schematic Progress
More progress on schematic. Image sensor schematic nearly finished, need
to check termination requirements of signals. Memory schematic nearly
solidified. LDO added to image sensor circuit for analog supply (3V).
Need to research termination requirements for memory as well. Need to
check what internal termination if any resistors are available in the
Zynq soc.
Connections:
- net labels removed: CTRL_SIG_BUS
Changed lines of the file:
@@
 	1    0    0    -1
 $EndComp
-Entry Bus Bus
-	2125 3925 2225 3825
-Entry Bus Bus
-	2125 4025 2225 3925
-Entry Bus Bus
-	2125 4125 2225 4025
-Entry Bus Bus
-	2125 4225 2225 4125
-Entry Bus Bus
-	2125 4325 2225 4225
-Entry Bus Bus
-	2125 4675 2225 4575
-Entry Bus Bus
-	2125 4775 2225 4675
-Entry Bus Bus
-	2125 4875 2225 4775
-Entry Bus Bus
-	2125 4475 2225 4375
-Text HLabel 1225 5050 0    60   BiDi ~ 0
-CTRL_SIG_BUS
 $Comp
 L ERJ-2RKF2400X R?
@@
 	1    0    0    -1
 $EndComp
-Entry Bus Bus
-	9450 2975 9550 3075
-Entry Bus Bus
-	9450 2875 9550 2975
 $Comp
 L ERA-2AEB510X R?
@@
 	1    0    0    -1
 $EndComp
-Entry Bus Bus
-	9450 3225 9550 3325
-Entry Bus Bus
-	9450 3125 9550 3225
 $Comp
 L ERA-2AEB510X R?
@@
 Wire Wire Line
 	4875 4775 4175 4775
-Wire Bus Line
-	2125 3925 2125 5050
-Wire Bus Line
-	3100 5050 1200 5050
 Wire Wire Line
 	6525 3475 6600 3475
@@
 Wire Wire Line
 	7550 3225 9450 3225
-Wire Bus Line
-	9550 2975 9550 5050
-Wire Bus Line
-	9550 5050 3075 5050
 Connection ~ 2025 5500
-Wire Bus Line
-	9550 3325 9550 3300
 Text Label 8475 1925 0    60   ~ 0
 DDR3L_D0
