File: PCB/OV7725_cam.sch (KiCad schematic (older format))
At the start: 32 parts

Commit message: Schematic Progress
More progress on schematic. Image sensor schematic nearly finished, need
to check termination requirements of signals. Memory schematic nearly
solidified. LDO added to image sensor circuit for analog supply (3V).
Need to research termination requirements for memory as well. Need to
check what internal termination if any resistors are available in the
Zynq soc.
Parts:
- removed C? (x5): CL05B104JP5NNNC, PCB_Footprints:C0402, symbol CL05B104JP5NNNC
- removed C? (x2): CL21A226KQQNNNE, PCB_Footprints:C0805, symbol CL21A226KQQNNNE
- removed FB?: BLM15HG601SN1D, PCB_Footprints:BLM15HG601SN1D, symbol BLM15HG601SN1D
- removed R?: RC1005F103CS, PCB_Footprints:R0402, symbol RC1005F103CS
- removed R? (x2): RC1005F472CS, PCB_Footprints:R0402, symbol RC1005F472CS
- removed R? (x18): ERA-2AEB510X, PCB_Footprints:R0402, symbol ERA-2AEB510X
- removed U?: OV07725-V28A, PCB_Footprints:OV07725-V28A, symbol OV07725-V28A
- added C? (x12): CL05B104JP5NNNC, PCB_Footprints:C0402, symbol CL05B104JP5NNNC
- added U? (x2): OV04689-H67A, PCB_Footprints:OV04689-H67A, symbol OV04689-H67A
Connections:
- net labels removed: CAM_D0, CAM_D1, CAM_D2, CAM_D3, CAM_D4, CAM_D5, CAM_D6, CAM_D7, CAM_D8, CAM_D9, CAM_D[1..10], VDDA
- wire segments 71 -> 10
Other:
- moved on the sheet: C?, LENS?
